File: Hardware/PMOD_buffer/PMOD_buffer.kicad_sch (KiCad schematic)
At the start: 42 parts, among them J1 Conn_Coaxial, J2 Conn_Coaxial, J3 Conn_Coaxial, J4 Conn_Coaxial, J5 Conn_Coaxial, J6 Conn_Coaxial, J7 Conn_Coaxial, J8 Conn_Coaxial, J9 Conn_02x06_Top_Bottom, U1 74LVC04AT14-13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

Commit message: Routing Board
Parts:
- added H1, H2, H3, H4: MountingHole_Pad, _tim-Mounting-Holes:4-40_Hole_Pad, symbol Mechanical:MountingHole_Pad
Connections:
- net GND: now also H1.1, H2.1, H3.1, H4.1

Commit message: Updating PMOD Buffer BOM
Parts:
- C1, C2, C3, C4: Digikey (none) -> 478-KGM21NR71H104KTCT-ND; MPN (none) -> KGM21NR71H104KT; Manufacturer (none) -> KYOCERA AVX
- C5: symbol Device:C_Polarized_Small_US -> Device:C_Small; Digikey (none) -> 1276-6455-1-ND; MPN (none) -> CL21A106KOQNNNG; Manufacturer (none) -> Samsung Electro-Mechanics
- J1, J2, J3, J4, J5, J6, J7, J8: value Conn_Coaxial -> RF2-152-T-00-50-G-HDW; MPN (none) -> RF2-152-T-00-50-G-HDW; Manufacturer (none) -> Adam Tech
- J9: value Conn_02x06_Top_Bottom -> 77313-101-12LF; Digikey (none) -> 609-5695-ND; MPN (none) -> 77313-101-12LF; Manufacturer (none) -> Amphenol ICC (FCI)
- R1, R13, R14, R19, R2, R20, R7, R8: Digikey (none) -> 541-3976-1-ND; MPN (none) -> CRCW080510K0FKEAC; Manufacturer (none) -> Vishay Dale
- R10, R11, R12, R15, R16, R17, R18, R21, R22, R23, R24, R3, R4, R5, R6, R9: Digikey (none) -> RMCF0805FT100RCT-ND; MPN (none) -> RMCF0805FT100R; Manufacturer (none) -> Stackpole Electronics Inc
- U1, U2, U3, U4: Digikey (none) -> 31-74LVC04AT14-13CT-ND; MPN (none) -> 74LVC04AT14-13; Manufacturer (none) -> Diodes Incorporated

Commit message: Generating Gerbers for Buffer
Other:
- moved on the sheet: R1, U1D
Changed lines of the file:
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@@
 	)
 	(junction
+		(at 55.88 54.61)
+		(diameter 0)
+		(color 0 0 0 0)
+	)
+	(junction
 		(at 172.72 101.6)
 		(diameter 0)
@@
 	)
 	(junction
-		(at 33.02 63.5)
+		(at 33.02 54.61)
 		(diameter 0)
 		(color 0 0 0 0)
@@
 	)
 	(junction
-		(at 55.88 63.5)
-		(diameter 0)
-		(color 0 0 0 0)
-	)
-	(junction
 		(at 86.36 101.6)
 		(diameter 0)
@@
 	(wire
 		(pts
-			(xy 55.88 54.61) (xy 55.88 63.5)
+			(xy 55.88 54.61) (xy 55.88 72.39)
 		)
 		(stroke
@@
 	(wire
 		(pts
-			(xy 34.29 63.5) (xy 33.02 63.5)
+			(xy 34.29 54.61) (xy 33.02 54.61)
 		)
 		(stroke
@@
 	(wire
 		(pts
-			(xy 27.94 63.5) (xy 33.02 63.5)
+			(xy 27.94 54.61) (xy 33.02 54.61)
 		)
 		(stroke
@@
 	(wire
 		(pts
-			(xy 33.02 63.5) (xy 33.02 64.77)
+			(xy 33.02 54.61) (xy 33.02 55.88)
 		)
 		(stroke
@@
 	(wire
 		(pts
-			(xy 55.88 63.5) (xy 55.88 72.39)
-		)
-		(stroke
-			(width 0)
-			(type default)
-		)
-	)
-	(wire
-		(pts
 			(xy 195.58 72.39) (xy 199.39 72.39)
 		)
@@
 	(wire
 		(pts
-			(xy 33.02 69.85) (xy 33.02 71.12)
+			(xy 33.02 60.96) (xy 33.02 62.23)
 		)
 		(stroke
@@
 	(wire
 		(pts
-			(xy 49.53 63.5) (xy 55.88 63.5)
+			(xy 49.53 54.61) (xy 55.88 54.61)
 		)
 		(stroke
@@
 	(global_label "PMOD_ja_2"
 		(shape input)
-		(at 27.94 63.5 180)
+		(at 27.94 54.61 180)
 		(fields_autoplaced yes)
 		(effects
@@
 		)
 		(property "Intersheetrefs" "${INTERSHEET_REFS}"
-			(at 14.7344 63.5 0)
+			(at 14.7344 54.61 0)
 			(effects
 				(font
@@
 	(symbol
 		(lib_id "74xx:74LS04")
-		(at 41.91 63.5 0)
+		(at 41.91 54.61 0)
 		(unit 4)
 		(exclude_from_sim no)
@@
 		(fields_autoplaced yes)
 		(property "Reference" "U1"
-			(at 41.91 54.61 0)
+			(at 41.91 45.72 0)
 			(effects
 				(font
@@
 		)
 		(property "Value" "74LVC04AT14-13"
-			(at 41.91 57.15 0)
+			(at 41.91 48.26 0)
 			(effects
 				(font
@@
 		)
 		(property "Footprint" "Package_SO:TSSOP-14_4.4x5mm_P0.65mm"
-			(at 41.91 63.5 0)
+			(at 41.91 54.61 0)
 			(effects
 				(font
@@
 		)
 		(property "Datasheet" "http://www.ti.com/lit/gpn/sn74LS04"
-			(at 41.91 63.5 0)
+			(at 41.91 54.61 0)
 			(effects
 				(font
@@
 		)
 		(property "Description" "IC INVERTER 6CH 6-INP 14TSSOP"
-			(at 41.91 63.5 0)
+			(at 41.91 54.61 0)
 			(effects
 				(font
@@
 		)
 		(property "Digikey" "31-74LVC04AT14-13CT-ND"
-			(at 41.91 63.5 0)
+			(at 41.91 54.61 0)
 			(effects
 				(font
@@
 		)
 		(property "MPN" "74LVC04AT14-13"
-			(at 41.91 63.5 0)
+			(at 41.91 54.61 0)
 			(effects
 				(font
@@
 		)
 		(property "Manufacturer" "Diodes Incorporated"
-			(at 41.91 63.5 0)
+			(at 41.91 54.61 0)
 			(effects
 				(font
@@
 	(symbol
 		(lib_id "power:GND")
-		(at 33.02 71.12 0)
+		(at 33.02 62.23 0)
 		(unit 1)
 		(exclude_from_sim no)
@@
 		(dnp no)
 		(property "Reference" "#PWR01"
-			(at 33.02 77.47 0)
+			(at 33.02 68.58 0)
 			(effects
 				(font
@@
 		)
 		(property "Value" "GND"
-			(at 33.02 74.93 0)
+			(at 33.02 66.04 0)
 			(effects
 				(font
@@
 		)
 		(property "Footprint" ""
-			(at 33.02 71.12 0)
+			(at 33.02 62.23 0)
 			(effects
 				(font
@@
 		)
 		(property "Datasheet" ""
-			(at 33.02 71.12 0)
+			(at 33.02 62.23 0)
 			(effects
 				(font
@@
 		)
 		(property "Description" "Power symbol creates a global label with name \"GND\" , ground"
-			(at 33.02 71.12 0)
+			(at 33.02 62.23 0)
 			(effects
 				(font
@@
 	(symbol
 		(lib_id "Device:R_Small_US")
-		(at 33.02 67.31 0)
+		(at 33.02 58.42 0)
 		(unit 1)
 		(exclude_from_sim no)
@@
 		(dnp no)
 		(property "Reference" "R1"
-			(at 28.194 66.04 0)
+			(at 28.194 57.15 0)
 			(effects
 				(font
@@
 		)
 		(property "Value" "10k"
-			(at 27.94 68.58 0)
+			(at 27.94 59.69 0)
 			(effects
 				(font
@@
 		)
 		(property "Footprint" "Resistor_SMD:R_0805_2012Metric"
-			(at 33.02 67.31 0)
+			(at 33.02 58.42 0)
 			(effects
 				(font
@@
 		)
 		(property "Datasheet" "~"
-			(at 33.02 67.31 0)
+			(at 33.02 58.42 0)
 			(effects
 				(font
@@
 		)
 		(property "Description" "RES 10K OHM 1% 1/8W 0805"
-			(at 33.02 67.31 0)
+			(at 33.02 58.42 0)
 			(effects
 				(font
@@
 		)
 		(property "Digikey" "541-3976-1-ND"
-			(at 33.02 67.31 0)
+			(at 33.02 58.42 0)
 			(effects
 				(font
@@
 		)
 		(property "MPN" "CRCW080510K0FKEAC"
-			(at 33.02 67.31 0)
+			(at 33.02 58.42 0)
 			(effects
 				(font
@@
 		)
 		(property "Manufacturer" "Vishay Dale"
-			(at 33.02 67.31 0)
+			(at 33.02 58.42 0)
 			(effects
 				(font
